Commit message: curved trajectory

File: config/combined.xacro (robot description, xacro)
@@ -1,8 +1,4 @@
-<?xml version="1.0" ?>
-<!-- =================================================================================== -->
-<!-- |    This document was autogenerated by xacro from /home/shanoj/catkin_ws/src/cooking_robot/urdf/primary_manipulator.xacro | -->
-<!-- |    EDITING THIS FILE BY HAND IS NOT RECOMMENDED                                 | -->
-<!-- =================================================================================== -->
-<robot name="primary_manipulator">
+<?xml version="1.0"?>
+<robot xmlns:xacro="http://www.ros.org/wiki/xacro" name="dual_manipulator">
     <material name="silver">
         <color rgba="0.700 0.700 0.700 1.000" />
@@ -411,3 +407,210 @@
         <!-- <mimic joint= 'joint_gripper_left' multiplier='-1' offset='0'/> -->
     </joint>
+    <material name="silver">
+        <color rgba="0.700 0.700 0.700 1.000" />
+    </material>
+    <transmission name="Revolute 1_tran">
+        <type>transmission_interface/SimpleTransmission</type>
+        <joint name="joint_1">
+            <hardwareInterface>hardware_interface/PositionJointInterface</hardwareInterface>
+        </joint>
+        <actuator name="Revolute 1_actr">
+            <hardwareInterface>hardware_interface/PositionJointInterface</hardwareInterface>
+            <mechanicalReduction>1</mechanicalReduction>
+        </actuator>
+    </transmission>
+    <transmission name="Revolute 2_tran">
+        <type>transmission_interface/SimpleTransmission</type>
+        <joint name="joint_2">
+            <hardwareInterface>hardware_interface/PositionJointInterface</hardwareInterface>
+        </joint>
+        <actuator name="Revolute 2_actr">
+            <hardwareInterface>hardware_interface/PositionJointInterface</hardwareInterface>
+            <mechanicalReduction>1</mechanicalReduction>
+        </actuator>
+    </transmission>
+    <transmission name="Revolute 3_tran">
+        <type>transmission_interface/SimpleTransmission</type>
+        <joint name="joint_3">
+            <hardwareInterface>hardware_interface/PositionJointInterface</hardwareInterface>
+        </joint>
+        <actuator name="Revolute 3_actr">
+            <hardwareInterface>hardware_interface/PositionJointInterface</hardwareInterface>
+            <mechanicalReduction>1</mechanicalReduction>
+        </actuator>
+    </transmission>
+    <transmission name="Revolute 4_tran">
+        <type>transmission_interface/SimpleTransmission</type>
+        <joint name="joint_4">
+            <hardwareInterface>hardware_interface/PositionJointInterface</hardwareInterface>
+        </joint>
+        <actuator name="Revolute 4_actr">
+            <hardwareInterface>hardware_interface/PositionJointInterface</hardwareInterface>
+            <mechanicalReduction>1</mechanicalReduction>
+        </actuator>
+    </transmission>
+    <gazebo reference="base_link1">
+        <material>Gazebo/Silver</material>
+        <mu1>0.2</mu1>
+        <mu2>0.2</mu2>
+        <selfCollide>true</selfCollide>
+        <gravity>true</gravity>
+    </gazebo>
+    <gazebo reference="link_1">
+        <material>Gazebo/Silver</material>
+        <mu1>0.2</mu1>
+        <mu2>0.2</mu2>
+        <selfCollide>true</selfCollide>
+    </gazebo>
+    <gazebo reference="link_2">
+        <material>Gazebo/Silver</material>
+        <mu1>0.2</mu1>
+        <mu2>0.2</mu2>
+        <selfCollide>true</selfCollide>
+    </gazebo>
+    <gazebo reference="link_3">
+        <material>Gazebo/Silver</material>
+        <mu1>0.2</mu1>
+        <mu2>0.2</mu2>
+        <selfCollide>true</selfCollide>
+    </gazebo>
+    <gazebo reference="stirrer_1">
+        <material>Gazebo/Silver</material>
+        <mu1>0.2</mu1>
+        <mu2>0.2</mu2>
+        <selfCollide>true</selfCollide>
+    </gazebo>
+    <link name="base_link1">
+        <inertial>
+            <origin rpy="0 0 0" xyz="4.5783389446227103e-05 -3.423407307852904e-11 0.041067543670996916" />
+            <mass value="2.090196446361125" />
+            <inertia ixx="0.006099" ixy="0.0" ixz="-2e-06" iyy="0.006106" iyz="0.0" izz="0.009727" />
+        </inertial>
+        <visual>
+            <origin rpy="0 0 0" xyz="0 0 0" />
+            <geometry>
+                <mesh filename="package://secondary_manipulator_3DoF_description/meshes/base_link.stl" scale="0.001 0.001 0.001" />
+            </geometry>
+            <material name="silver" />
+        </visual>
+        <collision>
+            <origin rpy="0 0 0" xyz="0 0 0" />
+            <geometry>
+                <mesh filename="package://secondary_manipulator_3DoF_description/meshes/base_link.stl" scale="0.001 0.001 0.001" />
+            </geometry>
+        </collision>
+    </link>
+    <joint name="j1" type="fixed">
+        <parent link="world" />
+        <child link="base_link1" />
+        <origin rpy="0.1 0.0 0.0" xyz="0.0 5.0 0.0" />
+    </joint>
+    <link name="link_1">
+        <inertial>
+            <origin rpy="0 0 0" xyz="-0.024369195599205848 -0.0013666751072870173 0.047358636153761555" />
+            <mass value="5.644227628176214" />
+            <inertia ixx="0.009655" ixy="-0.000472" ixz="0.00573" iyy="0.016996" iyz="0.000379" izz="0.013045" />
+        </inertial>
+        <visual>
+            <origin rpy="0 0 0" xyz="-0.0 -0.0 -0.07" />
+            <geometry>
+                <mesh filename="package://secondary_manipulator_3DoF_description/meshes/link_1_1.stl" scale="0.001 0.001 0.001" />
+            </geometry>
+            <material name="silver" />
+        </visual>
+        <collision>
+            <origin rpy="0 0 0" xyz="-0.0 -0.0 -0.07" />
+            <geometry>
+                <mesh filename="package://secondary_manipulator_3DoF_description/meshes/link_1_1.stl" scale="0.001 0.001 0.001" />
+            </geometry>
+        </collision>
+    </link>
+    <link name="link_2">
+        <inertial>
+            <origin rpy="0 0 0" xyz="-0.08155205936318585 -0.032554744515919276 -5.292016824753887e-12" />
+            <mass value="4.39179773511368" />
+            <inertia ixx="0.002102" ixy="0.00024" ixz="0.0" iyy="0.02561" iyz="0.0" izz="0.024791" />
+        </inertial>
+        <visual>
+            <origin rpy="0 0 0" xyz="0.09 0.015 -0.17" />
+            <geometry>
+                <mesh filename="package://secondary_manipulator_3DoF_description/meshes/link_2_1.stl" scale="0.001 0.001 0.001" />
+            </geometry>
+            <material name="silver" />
+        </visual>
+        <collision>
+            <origin rpy="0 0 0" xyz="0.09 0.015 -0.17" />
+            <geometry>
+                <mesh filename="package://secondary_manipulator_3DoF_description/meshes/link_2_1.stl" scale="0.001 0.001 0.001" />
+            </geometry>
+        </collision>
+    </link>
+    <link name="link_3">
+        <inertial>
+            <origin rpy="0 0 0" xyz="-0.002983021687897325 0.045124600240760884 -6.946881125902138e-10" />
+            <mass value="0.49113740866976063" />
+            <inertia ixx="0.000449" ixy="2e-06" ixz="0.0" iyy="0.00017" iyz="0.0" izz="0.000502" />
+        </inertial>
+        <visual>
+            <origin rpy="0 0 0" xyz="0.29 0.029 -0.17" />
+            <geometry>
+                <mesh filename="package://secondary_manipulator_3DoF_description/meshes/link_3_1.stl" scale="0.001 0.001 0.001" />
+            </geometry>
+            <material name="silver" />
+        </visual>
+        <collision>
+            <origin rpy="0 0 0" xyz="0.29 0.029 -0.17" />
+            <geometry>
+                <mesh filename="package://secondary_manipulator_3DoF_description/meshes/link_3_1.stl" scale="0.001 0.001 0.001" />
+            </geometry>
+        </collision>
+    </link>
+    <link name="stirrer_1">
+        <inertial>
+            <origin rpy="0 0 0" xyz="-0.12113338454910044 2.1163626406917047e-16 2.7755575615628914e-17" />
+            <mass value="2.0034028595901017" />
+            <inertia ixx="0.002813" ixy="-0.0" ixz="-0.0" iyy="0.007095" iyz="0.0" izz="0.009747" />
+        </inertial>
+        <visual>
+            <origin rpy="0 0 0" xyz="0.315 -0.0185 -0.17" />
+            <geometry>
+                <mesh filename="package://secondary_manipulator_3DoF_description/meshes/stirrer_1.stl" scale="0.001 0.001 0.001" />
+            </geometry>
+            <material name="silver" />
+        </visual>
+        <collision>
+            <origin rpy="0 0 0" xyz="0.315 -0.0185 -0.17" />
+            <geometry>
+                <mesh filename="package://secondary_manipulator_3DoF_description/meshes/stirrer_1.stl" scale="0.001 0.001 0.001" />
+            </geometry>
+        </collision>
+    </link>
+    <joint name="joint_1" type="revolute">
+        <origin rpy="0 0 0" xyz="0.0 0.0 0.07" />
+        <parent link="base_link1" />
+        <child link="link_1" />
+        <axis xyz="0.0 0.0 -1.0" />
+        <limit effort="100" lower="-1.0" upper="4.0" velocity="100" />
+    </joint>
+    <joint name="joint_2" type="revolute">
+        <origin rpy="0 0 0" xyz="-0.09 -0.015 0.1" />
+        <parent link="link_1" />
+        <child link="link_2" />
+        <axis xyz="0.0 -1.0 0.0" />
+        <limit effort="100" lower="-1.0" upper="4.0" velocity="100" />
+    </joint>
+    <joint name="joint_3" type="revolute">
+        <origin rpy="0 0 0" xyz="-0.2 -0.014 0.0" />
+        <parent link="link_2" />
+        <child link="link_3" />
+        <axis xyz="0.0 -1.0 0.0" />
+        <limit effort="100" lower="-1.0" upper="4.0" velocity="100" />
+    </joint>
+    <joint name="joint_4" type="revolute">
+        <origin rpy="0 0 0" xyz="-0.025 0.0475 0.0" />
+        <parent link="link_3" />
+        <child link="stirrer_1" />
+        <axis xyz="1.0 0.0 -0.0" />
+        <limit effort="100" lower="-1.0" upper="4.0" velocity="100" />
+    </joint>
 </robot>
